File: src/protectionCircuit.kicad_sch (KiCad schematic)
At the start: 20 parts, among them M1 CSD19534Q5A, M2 CSD19534Q5A, U1 LM74910QRGERQ1

Commit message: Tweaked a lot stuff
Parts:
- gave numbers to parts that had none: 1
- renumbered C_dvdt to C_dvdt1, Ccap to Ccap1, Ccs+ to Ccs+1, Cout to Cout1, Cscp to Cscp1, Ctmr to Ctmr1, Cuv to Cuv1, Cvin to Cvin1, Cvs to Cvs1, R_ILIM to R_ILIM1, R_ISCP to R_ISCP1, Rset to Rset1
Changed lines of the file:
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@@
 		(instances
 			(project "powerDristributionBoard"
-				(path "/d5fc2ae9-f21d-48b0-bd61-912ade1f672f/decf1042-8545-4374-a825-63213b68d513"
+				(path "/501e9f3f-9bfa-47dd-b56d-5fd6974f0d03/decf1042-8545-4374-a825-63213b68d513"
 					(reference "R_div4")
 					(unit 1)
@@
 		(instances
 			(project "powerDristributionBoard"
-				(path "/d5fc2ae9-f21d-48b0-bd61-912ade1f672f/decf1042-8545-4374-a825-63213b68d513"
+				(path "/501e9f3f-9bfa-47dd-b56d-5fd6974f0d03/decf1042-8545-4374-a825-63213b68d513"
 					(reference "M1")
 					(unit 1)
@@
 		(dnp no)
 		(fields_autoplaced yes)
-		(property "Reference" "Cvs"
+		(property "Reference" "Cvs1"
 			(at 149.86 118.1162 0)
 			(show_name no)
@@
 		(instances
 			(project "powerDristributionBoard"
-				(path "/d5fc2ae9-f21d-48b0-bd61-912ade1f672f/decf1042-8545-4374-a825-63213b68d513"
-					(reference "Cvs")
+				(path "/501e9f3f-9bfa-47dd-b56d-5fd6974f0d03/decf1042-8545-4374-a825-63213b68d513"
+					(reference "Cvs1")
 					(unit 1)
 				)
@@
 		(dnp no)
 		(fields_autoplaced yes)
-		(property "Reference" "Ccap"
+		(property "Reference" "Ccap1"
 			(at 134.62 67.3035 0)
 			(show_name no)
@@
 		(instances
 			(project "powerDristributionBoard"
-				(path "/d5fc2ae9-f21d-48b0-bd61-912ade1f672f/decf1042-8545-4374-a825-63213b68d513"
-					(reference "Ccap")
+				(path "/501e9f3f-9bfa-47dd-b56d-5fd6974f0d03/decf1042-8545-4374-a825-63213b68d513"
+					(reference "Ccap1")
 					(unit 1)
 				)
@@
 		(instances
 			(project "powerDristributionBoard"
-				(path "/d5fc2ae9-f21d-48b0-bd61-912ade1f672f/decf1042-8545-4374-a825-63213b68d513"
+				(path "/501e9f3f-9bfa-47dd-b56d-5fd6974f0d03/decf1042-8545-4374-a825-63213b68d513"
 					(reference "M2")
 					(unit 1)
@@
 		(instances
 			(project "powerDristributionBoard"
-				(path "/d5fc2ae9-f21d-48b0-bd61-912ade1f672f/decf1042-8545-4374-a825-63213b68d513"
+				(path "/501e9f3f-9bfa-47dd-b56d-5fd6974f0d03/decf1042-8545-4374-a825-63213b68d513"
 					(reference "#PWR033")
 					(unit 1)
@@
 		(instances
 			(project "powerDristributionBoard"
-				(path "/d5fc2ae9-f21d-48b0-bd61-912ade1f672f/decf1042-8545-4374-a825-63213b68d513"
+				(path "/501e9f3f-9bfa-47dd-b56d-5fd6974f0d03/decf1042-8545-4374-a825-63213b68d513"
 					(reference "#PWR031")
 					(unit 1)
@@
 		(dnp no)
 		(fields_autoplaced yes)
-		(property "Reference" "Ctmr"
+		(property "Reference" "Ctmr1"
 			(at 45.72 114.3062 0)
 			(show_name no)
@@
 		(instances
 			(project "powerDristributionBoard"
-				(path "/d5fc2ae9-f21d-48b0-bd61-912ade1f672f/decf1042-8545-4374-a825-63213b68d513"
-					(reference "Ctmr")
+				(path "/501e9f3f-9bfa-47dd-b56d-5fd6974f0d03/decf1042-8545-4374-a825-63213b68d513"
+					(reference "Ctmr1")
 					(unit 1)
 				)
@@
 		(instances
 			(project "powerDristributionBoard"
-				(path "/d5fc2ae9-f21d-48b0-bd61-912ade1f672f/decf1042-8545-4374-a825-63213b68d513"
+				(path "/501e9f3f-9bfa-47dd-b56d-5fd6974f0d03/decf1042-8545-4374-a825-63213b68d513"
 					(reference "R_div2")
 					(unit 1)
@@
 		(dnp no)
 		(fields_autoplaced yes)
-		(property "Reference" "C_dvdt"
+		(property "Reference" "C_dvdt1"
 			(at 185.42 118.1162 0)
 			(show_name no)
@@
 		(instances
 			(project "powerDristributionBoard"
-				(path "/d5fc2ae9-f21d-48b0-bd61-912ade1f672f/decf1042-8545-4374-a825-63213b68d513"
-					(reference "C_dvdt")
+				(path "/501e9f3f-9bfa-47dd-b56d-5fd6974f0d03/decf1042-8545-4374-a825-63213b68d513"
+					(reference "C_dvdt1")
 					(unit 1)
 				)
@@
 		(instances
 			(project "powerDristributionBoard"
-				(path "/d5fc2ae9-f21d-48b0-bd61-912ade1f672f/decf1042-8545-4374-a825-63213b68d513"
+				(path "/501e9f3f-9bfa-47dd-b56d-5fd6974f0d03/decf1042-8545-4374-a825-63213b68d513"
 					(reference "#PWR030")
 					(unit 1)
@@
 		(instances
 			(project "powerDristributionBoard"
-				(path "/d5fc2ae9-f21d-48b0-bd61-912ade1f672f/decf1042-8545-4374-a825-63213b68d513"
+				(path "/501e9f3f-9bfa-47dd-b56d-5fd6974f0d03/decf1042-8545-4374-a825-63213b68d513"
 					(reference "#PWR027")
 					(unit 1)
@@
 		(dnp no)
 		(fields_autoplaced yes)
-		(property "Reference" "Cscp"
+		(property "Reference" "Cscp1"
 			(at 173.9963 85.09 90)
 			(show_name no)
@@
 		(instances
 			(project "powerDristributionBoard"
-				(path "/d5fc2ae9-f21d-48b0-bd61-912ade1f672f/decf1042-8545-4374-a825-63213b68d513"
-					(reference "Cscp")
+				(path "/501e9f3f-9bfa-47dd-b56d-5fd6974f0d03/decf1042-8545-4374-a825-63213b68d513"
+					(reference "Cscp1")
 					(unit 1)
 				)
@@
 		(dnp no)
 		(fields_autoplaced yes)
-		(property "Reference" "Cuv"
+		(property "Reference" "Cuv1"
 			(at 91.44 163.8362 0)
 			(show_name no)
@@
 		(instances
 			(project "powerDristributionBoard"
-				(path "/d5fc2ae9-f21d-48b0-bd61-912ade1f672f/decf1042-8545-4374-a825-63213b68d513"
-					(reference "Cuv")
+				(path "/501e9f3f-9bfa-47dd-b56d-5fd6974f0d03/decf1042-8545-4374-a825-63213b68d513"
+					(reference "Cuv1")
 					(unit 1)
 				)
@@
 		(dnp no)
 		(fields_autoplaced yes)
-		(property "Reference" "Rset"
+		(property "Reference" "Rset1"
 			(at 167.64 62.2299 0)
 			(show_name no)
@@
 		(instances
 			(project "powerDristributionBoard"
-				(path "/d5fc2ae9-f21d-48b0-bd61-912ade1f672f/decf1042-8545-4374-a825-63213b68d513"
-					(reference "Rset")
+				(path "/501e9f3f-9bfa-47dd-b56d-5fd6974f0d03/decf1042-8545-4374-a825-63213b68d513"
+					(reference "Rset1")
 					(unit 1)
 				)
@@
 		(in_pos_files yes)
 		(dnp no)
-		(property "Reference" "R?"
+		(property "Reference" "R18"
 			(at 169.926 49.276 0)
 			(show_name no)
@@
 		(instances
 			(project "powerDristributionBoard"
-				(path "/d5fc2ae9-f21d-48b0-bd61-912ade1f672f/decf1042-8545-4374-a825-63213b68d513"
-					(reference "R?")
+				(path "/501e9f3f-9bfa-47dd-b56d-5fd6974f0d03/decf1042-8545-4374-a825-63213b68d513"
+					(reference "R18")
 					(unit 1)
 				)
@@
 		(dnp no)
 		(fields_autoplaced yes)
-		(property "Reference" "R_ISCP"
+		(property "Reference" "R_ISCP1"
 			(at 156.21 71.1199 0)
 			(show_name no)
@@
 		(instances
 			(project "powerDristributionBoard"
-				(path "/d5fc2ae9-f21d-48b0-bd61-912ade1f672f/decf1042-8545-4374-a825-63213b68d513"
-					(reference "R_ISCP")
+				(path "/501e9f3f-9bfa-47dd-b56d-5fd6974f0d03/decf1042-8545-4374-a825-63213b68d513"
+					(reference "R_ISCP1")
 					(unit 1)
 				)
@@
 		(dnp no)
 		(fields_autoplaced yes)
-		(property "Reference" "Cvin"
+		(property "Reference" "Cvin1"
 			(at 43.18 57.1562 0)
 			(show_name no)
@@
 		(instances
 			(project "powerDristributionBoard"
-				(path "/d5fc2ae9-f21d-48b0-bd61-912ade1f672f/decf1042-8545-4374-a825-63213b68d513"
-					(reference "Cvin")
+				(path "/501e9f3f-9bfa-47dd-b56d-5fd6974f0d03/decf1042-8545-4374-a825-63213b68d513"
+					(reference "Cvin1")
 					(unit 1)
 				)
@@
 		(dnp no)
 		(fields_autoplaced yes)
-		(property "Reference" "Cout"
+		(property "Reference" "Cout1"
 			(at 229.87 56.5149 0)
 			(show_name no)
@@
 		(instances
 			(project "powerDristributionBoard"
-				(path "/d5fc2ae9-f21d-48b0-bd61-912ade1f672f/decf1042-8545-4374-a825-63213b68d513"
-					(reference "Cout")
+				(path "/501e9f3f-9bfa-47dd-b56d-5fd6974f0d03/decf1042-8545-4374-a825-63213b68d513"
+					(reference "Cout1")
 					(unit 1)
 				)
@@
 		(dnp no)
 		(fields_autoplaced yes)
-		(property "Reference" "R_ILIM"
+		(property "Reference" "R_ILIM1"
 			(at 63.5 114.2999 0)
 			(show_name no)
@@
 		(instances
 			(project "powerDristributionBoard"
-				(path "/d5fc2ae9-f21d-48b0-bd61-912ade1f672f/decf1042-8545-4374-a825-63213b68d513"
-					(reference "R_ILIM")
+				(path "/501e9f3f-9bfa-47dd-b56d-5fd6974f0d03/decf1042-8545-4374-a825-63213b68d513"
+					(reference "R_ILIM1")
 					(unit 1)
 				)
@@
 		(instances
 			(project "powerDristributionBoard"
-				(path "/d5fc2ae9-f21d-48b0-bd61-912ade1f672f/decf1042-8545-4374-a825-63213b68d513"
+				(path "/501e9f3f-9bfa-47dd-b56d-5fd6974f0d03/decf1042-8545-4374-a825-63213b68d513"
 					(reference "R_div1")
 					(unit 1)
@@
 		(dnp no)
 		(fields_autoplaced yes)
-		(property "Reference" "Ccs+"
+		(property "Reference" "Ccs+1"
 			(at 173.9963 72.39 90)
 			(show_name no)
@@
 		(instances
 			(project "powerDristributionBoard"
-				(path "/d5fc2ae9-f21d-48b0-bd61-912ade1f672f/decf1042-8545-4374-a825-63213b68d513"
-					(reference "Ccs+")
+				(path "/501e9f3f-9bfa-47dd-b56d-5fd6974f0d03/decf1042-8545-4374-a825-63213b68d513"
+					(reference "Ccs+1")
 					(unit 1)
 				)
@@
 		(instances
 			(project "powerDristributionBoard"
-				(path "/d5fc2ae9-f21d-48b0-bd61-912ade1f672f/decf1042-8545-4374-a825-63213b68d513"
+				(path "/501e9f3f-9bfa-47dd-b56d-5fd6974f0d03/decf1042-8545-4374-a825-63213b68d513"
 					(reference "#PWR032")
 					(unit 1)
@@
 		(instances
 			(project "powerDristributionBoard"
-				(path "/d5fc2ae9-f21d-48b0-bd61-912ade1f672f/decf1042-8545-4374-a825-63213b68d513"
+				(path "/501e9f3f-9bfa-47dd-b56d-5fd6974f0d03/decf1042-8545-4374-a825-63213b68d513"
 					(reference "U1")
 					(unit 1)
@@
 		(instances
 			(project "powerDristributionBoard"
-				(path "/d5fc2ae9-f21d-48b0-bd61-912ade1f672f/decf1042-8545-4374-a825-63213b68d513"
+				(path "/501e9f3f-9bfa-47dd-b56d-5fd6974f0d03/decf1042-8545-4374-a825-63213b68d513"
 					(reference "#PWR028")
 					(unit 1)
@@
 		(instances
 			(project "powerDristributionBoard"
-				(path "/d5fc2ae9-f21d-48b0-bd61-912ade1f672f/decf1042-8545-4374-a825-63213b68d513"
+				(path "/501e9f3f-9bfa-47dd-b56d-5fd6974f0d03/decf1042-8545-4374-a825-63213b68d513"
 					(reference "R_div3")
 					(unit 1)
@@
 		(instances
 			(project "powerDristributionBoard"
-				(path "/d5fc2ae9-f21d-48b0-bd61-912ade1f672f/decf1042-8545-4374-a825-63213b68d513"
+				(path "/501e9f3f-9bfa-47dd-b56d-5fd6974f0d03/decf1042-8545-4374-a825-63213b68d513"
 					(reference "#PWR029")
 					(unit 1)

Commit message: Test MErge
Parts:
- added M3: CSD19534Q5A, powerDristributionBoard-import-fps:DQJ8, symbol Schlib1:CSD19534Q5A
Changed lines of the file:
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@@
+	)
+	(symbol
+		(lib_id "Schlib1:CSD19534Q5A")
+		(at 233.68 20.32 0)
+		(unit 1)
+		(body_style 1)
+		(exclude_from_sim no)
+		(in_bom yes)
+		(on_board yes)
+		(in_pos_files yes)
+		(dnp no)
+		(property "Reference" "M3"
+			(at 241.3 20.32 0)
+			(show_name no)
+			(do_not_autoplace no)
+			(effects
+				(font
+					(size 1.27 1.27)
+				)
+				(justify left bottom)
+			)
+		)
+		(property "Value" "CSD19534Q5A"
+			(at 241.3 35.56 0)
+			(show_name no)
+			(do_not_autoplace no)
+			(effects
+				(font
+					(size 1.27 1.27)
+				)
+				(justify left bottom)
+			)
+		)
+		(property "Footprint" "powerDristributionBoard-import-fps:DQJ8"
+			(at 233.68 20.32 0)
+			(hide yes)
+			(show_name no)
+			(do_not_autoplace no)
+			(effects
+				(font
+					(size 1.27 1.27)
+				)
+			)
+		)
+		(property "Datasheet" ""
+			(at 233.68 20.32 0)
+			(hide yes)
+			(show_name no)
+			(do_not_autoplace no)
+			(effects
+				(font
+					(size 1.27 1.27)
+				)
+			)
+		)
+		(property "Description" "100-V, N channel NexFETâ„¢ power MOSFET, single SON 5 mm x 6 mm, 15.1 mOhm 8-VSONP -55 to 150"
+			(at 233.68 20.32 0)
+			(hide yes)
+			(show_name no)
+			(do_not_autoplace no)
+			(effects
+				(font
+					(size 1.27 1.27)
+				)
+			)
+		)
+		(property "COPYRIGHT" "Copyright (C) 2026 Ultra Librarian. All rights reserved."
+			(at 233.68 20.32 0)
+			(hide yes)
+			(show_name no)
+			(do_not_autoplace no)
+			(effects
+				(font
+					(size 1.27 1.27)
+				)
+				(justify left bottom)
+			)
+		)
+		(property "MANUFACTURER_NAME" "Texas Instruments"
+			(at 233.68 20.32 0)
+			(hide yes)
+			(show_name no)
+			(do_not_autoplace no)
+			(effects
+				(font
+					(size 1.27 1.27)
+				)
+				(justify left bottom)
+			)
+		)
+		(property "MANUFACTURER_PART_NUMBER" "CSD19534Q5A"
+			(at 233.68 20.32 0)
+			(hide yes)
+			(show_name no)
+			(do_not_autoplace no)
+			(effects
+				(font
+					(size 1.27 1.27)
+				)
+				(justify left bottom)
+			)
+		)
+		(property "REFDES" "RefDes"
+			(at 254 7.62 0)
+			(hide yes)
+			(show_name no)
+			(do_not_autoplace no)
+			(effects
+				(font
+					(size 1.27 1.27)
+				)
+				(justify left bottom)
+			)
+		)
+		(property "TYPE" "Type"
+			(at 254 10.16 0)
+			(hide yes)
+			(show_name no)
+			(do_not_autoplace no)
+			(effects
+				(font
+					(size 1.27 1.27)
+				)
+				(justify left bottom)
+			)
+		)
+		(pin "4"
+		)
+		(pin "1"
+		)
+		(pin "2"
+		)
+		(pin "3"
+		)
+		(pin "5"
+		)
+		(pin "6"
+		)
+		(pin "7"
+		)
+		(pin "8"
+		)
+		(instances
+			(project "powerDristributionBoard"
+				(path "/501e9f3f-9bfa-47dd-b56d-5fd6974f0d03/decf1042-8545-4374-a825-63213b68d513"
+					(reference "M3")
+					(unit 1)
+				)
+			)
+		)
 	)
 	(symbol
