File: src/5V_Converter.kicad_sch (KiCad schematic)
At the start: 16 parts, among them U3 TPS566238RQFR

Commit message: Edited PCB layout
Parts:
- renumbered C37 to C36, C45 to C37, C47 to C39, C46 to C40, C48 to C41, C39 to C43, C40 to C44, C49 to C45, C50 to C46, C41 to C47, R15 to R17, R16 to R18
Changed lines of the file:
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@@
 		(dnp no)
 		(fields_autoplaced yes)
-		(property "Reference" "C48"
+		(property "Reference" "C41"
 			(at 137.1536 83.82 90)
 			(show_name no)
@@
 			(project "powerDristributionBoard"
 				(path "/501e9f3f-9bfa-47dd-b56d-5fd6974f0d03/f7fc7c23-3a4e-412b-b14d-71f85b15285a"
-					(reference "C48")
+					(reference "C41")
 					(unit 1)
 				)
@@
 		(dnp no)
 		(fields_autoplaced yes)
-		(property "Reference" "R16"
+		(property "Reference" "R18"
 			(at 171.45 111.7599 0)
 			(show_name no)
@@
 			(project "powerDristributionBoard"
 				(path "/501e9f3f-9bfa-47dd-b56d-5fd6974f0d03/f7fc7c23-3a4e-412b-b14d-71f85b15285a"
-					(reference "R16")
+					(reference "R18")
 					(unit 1)
 				)
@@
 		(dnp no)
 		(fields_autoplaced yes)
-		(property "Reference" "C37"
+		(property "Reference" "C36"
 			(at 39.37 104.1335 0)
 			(show_name no)
@@
 			(project "powerDristributionBoard"
 				(path "/501e9f3f-9bfa-47dd-b56d-5fd6974f0d03/f7fc7c23-3a4e-412b-b14d-71f85b15285a"
-					(reference "C37")
+					(reference "C36")
 					(unit 1)
 				)
@@
 		(dnp no)
 		(fields_autoplaced yes)
-		(property "Reference" "#PWR016"
+		(property "Reference" "#PWR025"
 			(at 105.41 137.16 0)
 			(hide yes)
@@
 			(project "powerDristributionBoard"
 				(path "/501e9f3f-9bfa-47dd-b56d-5fd6974f0d03/f7fc7c23-3a4e-412b-b14d-71f85b15285a"
-					(reference "#PWR016")
+					(reference "#PWR025")
 					(unit 1)
 				)
@@
 		(dnp no)
 		(fields_autoplaced yes)
-		(property "Reference" "C46"
+		(property "Reference" "C40"
 			(at 86.36 114.2935 0)
 			(show_name no)
@@
 			(project "powerDristributionBoard"
 				(path "/501e9f3f-9bfa-47dd-b56d-5fd6974f0d03/f7fc7c23-3a4e-412b-b14d-71f85b15285a"
-					(reference "C46")
+					(reference "C40")
 					(unit 1)
 				)
@@
 		(dnp no)
 		(fields_autoplaced yes)
-		(property "Reference" "C41"
+		(property "Reference" "C47"
 			(at 236.22 104.1335 0)
 			(show_name no)
@@
 			(project "powerDristributionBoard"
 				(path "/501e9f3f-9bfa-47dd-b56d-5fd6974f0d03/f7fc7c23-3a4e-412b-b14d-71f85b15285a"
-					(reference "C41")
+					(reference "C47")
 					(unit 1)
 				)
@@
 		(dnp no)
 		(fields_autoplaced yes)
-		(property "Reference" "C40"
+		(property "Reference" "C44"
 			(at 198.12 104.1335 0)
 			(show_name no)
@@
 			(project "powerDristributionBoard"
 				(path "/501e9f3f-9bfa-47dd-b56d-5fd6974f0d03/f7fc7c23-3a4e-412b-b14d-71f85b15285a"
-					(reference "C40")
+					(reference "C44")
 					(unit 1)
 				)
@@
 		(dnp no)
 		(fields_autoplaced yes)
-		(property "Reference" "C39"
+		(property "Reference" "C43"
 			(at 185.42 104.1335 0)
 			(show_name no)
@@
 			(project "powerDristributionBoard"
 				(path "/501e9f3f-9bfa-47dd-b56d-5fd6974f0d03/f7fc7c23-3a4e-412b-b14d-71f85b15285a"
-					(reference "C39")
+					(reference "C43")
 					(unit 1)
 				)
@@
 		(dnp no)
 		(fields_autoplaced yes)
-		(property "Reference" "C47"
+		(property "Reference" "C39"
 			(at 74.93 110.4835 0)
 			(show_name no)
@@
 			(project "powerDristributionBoard"
 				(path "/501e9f3f-9bfa-47dd-b56d-5fd6974f0d03/f7fc7c23-3a4e-412b-b14d-71f85b15285a"
-					(reference "C47")
+					(reference "C39")
 					(unit 1)
 				)
@@
 		(dnp no)
 		(fields_autoplaced yes)
-		(property "Reference" "C49"
+		(property "Reference" "C45"
 			(at 210.82 104.1335 0)
 			(show_name no)
@@
 			(project "powerDristributionBoard"
 				(path "/501e9f3f-9bfa-47dd-b56d-5fd6974f0d03/f7fc7c23-3a4e-412b-b14d-71f85b15285a"
-					(reference "C49")
+					(reference "C45")
 					(unit 1)
 				)
@@
 		(dnp no)
 		(fields_autoplaced yes)
-		(property "Reference" "C45"
+		(property "Reference" "C37"
 			(at 49.53 104.1335 0)
 			(show_name no)
@@
 			(project "powerDristributionBoard"
 				(path "/501e9f3f-9bfa-47dd-b56d-5fd6974f0d03/f7fc7c23-3a4e-412b-b14d-71f85b15285a"
-					(reference "C45")
+					(reference "C37")
 					(unit 1)
 				)
@@
 		(dnp no)
 		(fields_autoplaced yes)
-		(property "Reference" "R15"
+		(property "Reference" "R17"
 			(at 171.45 96.5199 0)
 			(show_name no)
@@
 			(project "powerDristributionBoard"
 				(path "/501e9f3f-9bfa-47dd-b56d-5fd6974f0d03/f7fc7c23-3a4e-412b-b14d-71f85b15285a"
-					(reference "R15")
+					(reference "R17")
 					(unit 1)
 				)
@@
 		(dnp no)
 		(fields_autoplaced yes)
-		(property "Reference" "C50"
+		(property "Reference" "C46"
 			(at 223.52 104.1335 0)
 			(show_name no)
@@
 			(project "powerDristributionBoard"
 				(path "/501e9f3f-9bfa-47dd-b56d-5fd6974f0d03/f7fc7c23-3a4e-412b-b14d-71f85b15285a"
-					(reference "C50")
-					(unit 1)
-				)
+					(reference "C46")
+					(unit 1)
+				)
