File: src/5V_Converter.kicad_sch (KiCad schematic)
At the start: 16 parts, among them U3 TPS566238RQFR

Commit message: GG
Other:
- moved on the sheet: C36, C37, C38, C39, C40, C41, C42, C43, C44, C45, C46, C47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

Commit message: Completed half of the PCB layout
Other:
- moved on the sheet: C36, C37, C38, C39, C40, C41, C42, C43, C44, C45, C46, C47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

Commit message: Upated parts and BOM
Parts:
- C36, C37, C43, C44, C45, C46: LCSC Part (none) -> C5677683; MPN (none) -> MSAST21GBB5226MTNC12; Manufacturer (none) -> Taiyo Yuden
- C38, C47: LCSC Part (none) -> C108079; MPN (none) -> CC0603KRX7R7BB104; Manufacturer (none) -> YAGEO
- C39: LCSC Part (none) -> C2180996; MPN (none) -> C0603C105Z8VACTU; Manufacturer (none) -> KEMET
- C40: LCSC Part (none) -> C85735; MPN (none) -> GRM155R71C103KA01D; Manufacturer (none) -> Murata Electronics
- C41: LCSC Part (none) -> C71629; MPN (none) -> GRM155R71C104KA88D; Manufacturer (none) -> Murata Electronics
- C42: LCSC Part (none) -> C513616; MPN (none) -> CC0201JRNPO8BN330; Manufacturer (none) -> YAGEO
- L2: LCSC Part (none) -> C5337632; MPN (none) -> DR125-2R2-R; Manufacturer (none) -> EATON
- R17: LCSC Part (none) -> C123420; MPN (none) -> RC0603FR-07220KL; Manufacturer (none) -> YAGEO
- R18: LCSC Part (none) -> C100001; MPN (none) -> RC0603FR-0730KL; Manufacturer (none) -> YAGEO
- U3: LCSC Part (none) -> C5219353; MPN (none) -> TPS566238RQFR; Manufacturer (none) -> Texas Instruments

Commit message: Updated BOM
Parts:
- C38, C47: value 0.1uf -> 100nf
Changed lines of the file:
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@@
 			)
 		)
-		(property "Value" "0.1uf"
+		(property "Value" "100nf"
 			(at 237.49 91.4335 0)
 			(show_name no)
@@
 			)
 		)
-		(property "Value" "0.1uf"
+		(property "Value" "100nf"
 			(at 63.5 91.4335 0)
 			(show_name no)

Commit message: Changed 5V inductor
Parts:
- L2: footprint PowerPCB_Footprints:DR125-2R2-R -> PowerPCB_Footprints:SPM6530T-1R5M100; LCSC Part C5337632 -> C76854; MPN DR125-2R2-R -> SPM6530T-1R5M100; Manufacturer EATON -> TDK
Changed lines of the file:
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@@
 			)
 		)
-		(property "Footprint" "PowerPCB_Footprints:DR125-2R2-R"
+		(property "Footprint" "PowerPCB_Footprints:SPM6530T-1R5M100"
 			(at 151.13 74.93 0)
 			(hide yes)
@@
 			)
 		)
-		(property "Datasheet" "https://www.lcsc.com/datasheet/C5337632.pdf?spm=wm.sxq.inf.ggs___wm.fly.bg.0.xh&lcsc_vid=RwAMXlJfTlBYBAYHElQKUVVQTwJbU10DRwVcX1VVEgQxVlNfRVlcX1RXRVJZXjsOAxUeFF5JWBYZEEoKFBINSQcJGk4NBhADEA4cHktXRllfSQwSGg0%3D"
+		(property "Datasheet" "https://jlcpcb.com/partdetail/TDK-SPM6530T1R5M100/C76854"
 			(at 151.13 74.93 0)
 			(hide yes)
@@
 			)
 		)
-		(property "LCSC Part" "C5337632"
+		(property "LCSC Part" "C76854"
 			(at 151.13 74.93 90)
 			(hide yes)
@@
 			)
 		)
-		(property "MPN" "DR125-2R2-R"
+		(property "MPN" "SPM6530T-1R5M100"
 			(at 151.13 74.93 90)
 			(hide yes)
@@
 			)
 		)
-		(property "Manufacturer" "EATON"
+		(property "Manufacturer" "TDK"
 			(at 151.13 74.93 90)
 			(hide yes)

Commit message: Changed inductors and updated BOM
Parts:
- L2: value 2.2uH -> 1.5uH
Changed lines of the file:
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@@
 			)
 		)
-		(property "Value" "2.2uH"
+		(property "Value" "1.5uH"
 			(at 151.13 72.39 90)
 			(show_name no)
