File: src/powerDristributionBoard.kicad_pcb (KiCad board)
At the start: 2 copper layers, 152.4 x 101.6 mm, 0 parts

Commit message: Finalized schematic
Parts:
- added C1: 4.7uf, Capacitor_SMD:C_1210_3225Metric, F.Cu at (201.1, 55.7)
- added C10: 10nf, Capacitor_SMD:C_0603_1608Metric, F.Cu at (188.2, 75.6)
- added C11: 10nf, Capacitor_SMD:C_0603_1608Metric, F.Cu at (188.2, 78.1)
- added C12: 10nf, Capacitor_SMD:C_0603_1608Metric, F.Cu at (188.2, 80.6)
- added C13: 1uf, Capacitor_SMD:C_0603_1608Metric, F.Cu at (188.2, 83.1)
- added C14: 4.7nf, Capacitor_SMD:C_0603_1608Metric, F.Cu at (192.2, 68.1)
- added C15: 68nf, Capacitor_SMD:C_0603_1608Metric, F.Cu at (192.2, 70.6)
- added C16: 47pf, Capacitor_SMD:C_0603_1608Metric, F.Cu at (192.2, 73.1)
- added C17: 1nf, Capacitor_SMD:C_0402_1005Metric, F.Cu at (211.1, 71.4)
- added C18: 100nf, Capacitor_SMD:C_0603_1608Metric, F.Cu at (192.2, 75.6)
- added C19: 100pf, Capacitor_SMD:C_0603_1608Metric, F.Cu at (192.2, 78.1)
- added C2: 4.7uf, Capacitor_SMD:C_1210_3225Metric, F.Cu at (201.1, 60.0)
- added C20: 2.2uf, Capacitor_SMD:C_0603_1608Metric, F.Cu at (192.2, 80.6)
- added C21: 22uf, Capacitor_SMD:C_1210_3225Metric, F.Cu at (206.8, 60.0)
- added C22: 22uf, Capacitor_SMD:C_1210_3225Metric, F.Cu at (206.8, 64.2)
- added C23: 22uf, Capacitor_SMD:C_1210_3225Metric, F.Cu at (206.8, 68.5)
- added C24: 22uf, Capacitor_SMD:C_1210_3225Metric, F.Cu at (206.8, 72.7)
- added C25: 22uf, Capacitor_SMD:C_0805_2012Metric, F.Cu at (201.6, 125.2)
- added C26: 22uf, Capacitor_SMD:C_0805_2012Metric, F.Cu at (201.6, 128.2)
- added C27: 100nf, Capacitor_SMD:C_0603_1608Metric, F.Cu at (205.8, 125.0)
- added C28: 1uf, Capacitor_SMD:C_0603_1608Metric, F.Cu at (205.8, 127.5)
- added C29: 10nf, Capacitor_SMD:C_0402_1005Metric, F.Cu at (213.6, 133.6)
- added C3: 4.7uf, Capacitor_SMD:C_1210_3225Metric, F.Cu at (201.1, 64.2)
- added C30: 100nf, Capacitor_SMD:C_0402_1005Metric, F.Cu at (213.6, 135.5)
- added C31: 33pf, Capacitor_SMD:C_0603_1608Metric, F.Cu at (205.8, 130.0)
- added C32: 22uf, Capacitor_SMD:C_0805_2012Metric, F.Cu at (201.6, 131.3)
- added C33: 22uf, Capacitor_SMD:C_0805_2012Metric, F.Cu at (201.6, 134.3)
- added C34: 22uf, Capacitor_SMD:C_0805_2012Metric, F.Cu at (201.6, 137.3)
- added C35: 22uf, Capacitor_SMD:C_0805_2012Metric, F.Cu at (201.6, 140.3)
- added C36: 100nf, Capacitor_SMD:C_0603_1608Metric, F.Cu at (205.8, 132.5)
- added C37: 22uf, Capacitor_SMD:C_0805_2012Metric, F.Cu at (85.3, 123.8)
- added C38: 0.1uf, Capacitor_SMD:C_0603_1608Metric, F.Cu at (105.1, 123.5)
- added C39: 22uf, Capacitor_SMD:C_0805_2012Metric, F.Cu at (85.3, 126.8)
- added C4: 4.7uf, Capacitor_SMD:C_1210_3225Metric, F.Cu at (201.1, 68.5)
- added C40: 22uf, Capacitor_SMD:C_0805_2012Metric, F.Cu at (85.3, 129.8)
- added C41: 0.1uf, Capacitor_SMD:C_0603_1608Metric, F.Cu at (105.1, 126.0)
- added C42: 33pf, Capacitor_SMD:C_0201_0603Metric, F.Cu at (92.6, 137.7)
- added C43: 100nf, Capacitor_SMD:C_0603_1608Metric, F.Cu at (192.2, 83.1)
- added C44: 100nf, Capacitor_SMD:C_0603_1608Metric, F.Cu at (196.2, 68.1)
- added C45: 22uf, Capacitor_SMD:C_0805_2012Metric, F.Cu at (85.3, 132.8)
- added C46: 10nf, Capacitor_SMD:C_0402_1005Metric, F.Cu at (104.5, 135.8)
- added C47: 1uf, Capacitor_SMD:C_0603_1608Metric, F.Cu at (105.1, 128.5)
- added C48: 100nf, Capacitor_SMD:C_0402_1005Metric, F.Cu at (104.5, 137.8)
- added C49: 22uf, Capacitor_SMD:C_0805_2012Metric, F.Cu at (85.3, 135.8)
- added C5: 4.7uf, Capacitor_SMD:C_1210_3225Metric, F.Cu at (201.1, 72.7)
- added C50: 22uf, Capacitor_SMD:C_0805_2012Metric, F.Cu at (85.3, 138.8)
- added C6: 4.7uf, Capacitor_SMD:C_1210_3225Metric, F.Cu at (206.8, 55.7)
- added C7: 10nf, Capacitor_SMD:C_0603_1608Metric, F.Cu at (188.2, 68.1)
- added C8: 10nf, Capacitor_SMD:C_0603_1608Metric, F.Cu at (188.2, 70.6)
- added C9: 10nf, Capacitor_SMD:C_0603_1608Metric, F.Cu at (188.2, 73.1)
- added CN1: XT90_PCB_Mount_Male, PowerPCB_Footprints:XT-90_PCB_Mount_Male, F.Cu at (137.4, 109.9)
- added CN2: XT30_PCB_Mount_Female, PowerPCB_Footprints:XT30_PCB_Mount_Female, F.Cu at (133.5, 77.1)
- added CN3: XT30_PCB_Mount_Female, PowerPCB_Footprints:XT30_PCB_Mount_Female, F.Cu at (148.2, 77.1)
- added CN4: XT30_PCB_Mount_Female, PowerPCB_Footprints:XT30_PCB_Mount_Female, F.Cu at (163.0, 77.1)
- added C_dvdt1: 10nf, Capacitor_SMD:C_0603_1608Metric, F.Cu at (82.1, 65.6)
- added Ccap1: 100nf, Capacitor_SMD:C_0603_1608Metric, F.Cu at (82.1, 68.1)
- added Ccs+1: 10nf, Capacitor_SMD:C_0603_1608Metric, F.Cu at (82.1, 70.6)
- added Ciscp1: 10nf, Capacitor_SMD:C_0603_1608Metric, F.Cu at (82.1, 73.1)
- added Cout1: 100uf, Capacitor_THT:CP_Radial_D7.5mm_P2.50mm, F.Cu at (95.6, 68.9)
- added Ctmr1: 68nf, Capacitor_SMD:C_0603_1608Metric, F.Cu at (82.1, 75.6)
- added Cuv1: 100nf, Capacitor_SMD:C_0603_1608Metric, F.Cu at (82.1, 78.2)
- added Cvin1: 100nf, Capacitor_SMD:C_1210_3225Metric, F.Cu at (96.8, 61.6)
- added Cvs1: 100nf, Capacitor_SMD:C_0603_1608Metric, F.Cu at (86.1, 65.6)
- added D1: SMAJ48CA, PowerPCB_Footprints:SMAJ48CA, F.Cu at (97.4, 57.5)
- added D2: LED, LED_SMD:LED_1206_3216Metric, F.Cu at (155.6, 98.1)
- added D3: LED, LED_SMD:LED_0603_1608Metric, F.Cu at (150.7, 97.7)
- added D5: LED, LED_SMD:LED_0603_1608Metric, F.Cu at (150.7, 100.2)
- added D6: PESD12VS1ULD-QYL, PowerPCB_Footprints:PESD12VS1ULD-QYL, F.Cu at (154.2, 100.8)
- added D7: USSD0571P6W, PowerPCB_Footprints:USSD0571P6W, F.Cu at (166.0, 97.6)
- added D8: ESD351DPYR, PowerPCB_Footprints:ESD351DPYR, F.Cu at (156.9, 100.7)
- added D9: LED(Red), LED_SMD:LED_0603_1608Metric, F.Cu at (150.7, 102.8)
- added F1: BSMD2920L-800-24V, PowerPCB_Footprints:BSMD2920L-800-24V, F.Cu at (153.9, 92.8)
- added L1: 6.8uH, PowerPCB_Footprints:SMTC1010A-6R8MT, F.Cu at (192.2, 60.2)
- added L2: 2.2uH, PowerPCB_Footprints:DR125-2R2-R, F.Cu at (95.3, 129.6)
- added L3: 1.8uH, PowerPCB_Footprints:XAL7070-182MEC, F.Cu at (212.1, 128.2)
- added M1: CSD19534Q5A, PowerPCB_Footprints:CSD19534Q5A, F.Cu at (83.9, 59.7)
- added M2: CSD19534Q5A, PowerPCB_Footprints:CSD19534Q5A, F.Cu at (90.8, 59.7)
- added M3: CSD19534Q5A, PowerPCB_Footprints:CSD19534Q5A, F.Cu at (213.4, 57.8)
- added M4: NTMFS4D5N08XT1G, PowerPCB_Footprints:NTMFS4D5N08XT1G, F.Cu at (210.1, 79.7)
- added R1: 22k 0.25W, Resistor_SMD:R_1206_3216Metric, F.Cu at (161.2, 98.0)
- added R10: 90.9k, Resistor_SMD:R_0805_2012Metric, F.Cu at (210.0, 134.1)
- added R11: 20k, Resistor_SMD:R_0805_2012Metric, F.Cu at (210.0, 137.0)
- added R15: 220k, Resistor_SMD:R_0603_1608Metric, F.Cu at (105.1, 131.0)
- added R16: 30k, Resistor_SMD:R_0603_1608Metric, F.Cu at (105.1, 133.6)
- added R17: Find Val, Resistor_SMD:R_0603_1608Metric, F.Cu at (150.7, 110.4)
- added R18: 5mOhms, PowerPCB_Footprints:CSNL2010, F.Cu at (96.0, 75.6)
- added R2: 59k, Resistor_SMD:R_0603_1608Metric, F.Cu at (196.2, 70.6)
- added R3: 9.76k, Resistor_SMD:R_0603_1608Metric, F.Cu at (196.2, 73.1)
- added R4: 2.15k, Resistor_SMD:R_0805_2012Metric, F.Cu at (211.8, 68.9)
- added R5: 100k, Resistor_SMD:R_0603_1608Metric, F.Cu at (196.2, 75.6)
- added R6: 49.9, Resistor_SMD:R_0603_1608Metric, F.Cu at (196.2, 78.1)
- added R7: Find Val, Resistor_SMD:R_0603_1608Metric, F.Cu at (150.7, 105.4)
- added R8: 5mOhms, PowerPCB_Footprints:CSNL2010, F.Cu at (202.2, 77.0)
- added R9: Find Val, Resistor_SMD:R_0603_1608Metric, F.Cu at (150.7, 107.9)
- added R_ILIM1: 20k 1%, Resistor_SMD:R_0603_1608Metric, F.Cu at (86.1, 68.1)
- added R_IMON1: 6.04k 1%, Resistor_SMD:R_0603_1608Metric, F.Cu at (86.1, 70.6)
- added R_ISCP1: 952 1%, Resistor_SMD:R_0603_1608Metric, F.Cu at (86.1, 73.1)
- added R_div1: 100k, Resistor_SMD:R_0603_1608Metric, F.Cu at (86.1, 75.6)
- added R_div2: 3.83k 1%, Resistor_SMD:R_0603_1608Metric, F.Cu at (86.1, 78.2)
- added R_div3: 100k, Resistor_SMD:R_0603_1608Metric, F.Cu at (90.1, 65.6)
- added R_div4: 1k 1%, Resistor_SMD:R_0603_1608Metric, F.Cu at (90.1, 68.1)
- added Rset1: 50 1%, Resistor_SMD:R_0603_1608Metric, F.Cu at (90.1, 70.6)
- added U1: LM74910QRGERQ1, PowerPCB_Footprints:LM74910QRGERQ1, F.Cu at (102.5, 76.1)
- added U2: LM5190RGYR_(20V-50V), PowerPCB_Footprints:LM5190RGYR, F.Cu at (213.0, 65.0)
- added U3: TPS566238RQFR, PowerPCB_Footprints:TPS566238RQFR, F.Cu at (89.7, 138.2)
- added U4: TPS566238RQFR, PowerPCB_Footprints:TPS566238RQFR, F.Cu at (214.4, 137.9)
Other:
- board size 152.4 x 101.6 mm -> 150 x 100 mm

Commit message: Edited PCB layout
Parts:
- moved C50 171.5 mm to (36.7, 153.6)
- moved C51 171.5 mm to (36.7, 156.1)
- moved C52 171.5 mm to (44.5, 162.2)
- moved C53 171.5 mm to (44.5, 164.2)
- moved C54 171.5 mm to (36.7, 158.6)
- moved C59 171.5 mm to (36.7, 161.2)
- moved C48 171.5 mm to (32.4, 153.9)
- moved C49 171.5 mm to (32.4, 156.9)
- moved C55 171.5 mm to (32.4, 159.9)
- moved C56 171.5 mm to (32.4, 162.9)
- moved C57 171.5 mm to (32.4, 165.9)
- moved C58 171.5 mm to (32.4, 168.9)
- moved L3 171.5 mm to (43.0, 156.8)
- moved R22 171.5 mm to (40.9, 162.7)
- moved R23 171.5 mm to (40.9, 165.6)
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- renumbered Cvin1 to C1, C43 to C10, C13 to C11, C15 to C12, C44 to C13, C16 to C14, C1 to C15, C14 to C16, C2 to C17, C17 to C18, C3 to C19, Ctmr1 to C2, C4 to C20, C5 to C21, C6 to C22, C7 to C23, C18 to C24, C20 to C25, C8 to C26, C9 to C27, C10 to C28, C19 to C29, Cuv1 to C3, C11 to C30, C12 to C31, C21 to C32, C22 to C33, C23 to C34, C24 to C35, C37 to C36, C45 to C37, C47 to C39, Ccap1 to C4, C46 to C40, C48 to C41, C39 to C43, C40 to C44, C49 to C45, C50 to C46, C41 to C47, C25 to C48, C26 to C49, Cvs1 to C5, C27 to C50, C28 to C51, C29 to C52, C30 to C53, C31 to C54, C32 to C55, C33 to C56, C34 to C57, C35 to C58, C36 to C59, Ccs+1 to C6, Ciscp1 to C7, C_dvdt1 to C8, Cout1 to C9, CN4 to CN3, CN3 to CN4, D5 to D3, D3 to D4, D9 to D5, D8 to D7, D7 to D8, R_IMON1 to R1, R3 to R10, R4 to R11, R2 to R12, R5 to R13, R6 to R14, R8 to R15, R1 to R16, R15 to R17, R16 to R18, R7 to R19, R_ILIM1 to R2, R9 to R20, R17 to R21, R10 to R22, R11 to R23, R_div3 to R3, R_div4 to R4, R_div1 to R5, R_div2 to R6, R_ISCP1 to R7, Rset1 to R8, R18 to R9

Commit message: Edited PCB layout
Parts:
- moved C15 75.0 mm to (236.8, 28.7)
- moved C17 75.0 mm to (238.6, 48.4)
- moved C20 75.0 mm to (248.6, 48.5)
- moved C21 75.0 mm to (253.6, 48.5)
- moved C23 75.0 mm to (241.1, 18.5)
- moved C24 75.0 mm to (233.6, 27.9)
- moved C26 75.0 mm to (243.6, 18.5)
- moved C27 75.0 mm to (246.1, 18.5)
- moved C28 75.0 mm to (248.6, 18.5)
- moved C30 75.0 mm to (251.1, 18.5)
- moved C31 75.0 mm to (253.6, 18.5)
- moved M4 75.0 mm to (243.7, 39.1)
- moved C10 75.0 mm to (225.1, 25.7)
- moved C11 75.0 mm to (231.4, 25.7)
- moved C12 75.0 mm to (222.6, 36.2)
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
Commit message: testing
Parts:
- moved C58 105.7 mm to (133.0, 136.4), turned to 90 degrees
- moved C57 101.9 mm to (130.0, 136.4), turned to 90 degrees
- moved C56 98.2 mm to (127.0, 136.4), turned to 90 degrees
- moved R23 96.5 mm to (129.7, 128.0), turned to 90 degrees
- moved U4 95.5 mm to (130.6, 123.6), turned to 90 degrees
- moved C55 94.5 mm to (124.0, 136.4), turned to 90 degrees
- moved C59 93.2 mm to (125.2, 132.2), turned to 90 degrees
- moved C53 92.7 mm to (128.2, 124.3), turned to 90 degrees
- moved R22 92.6 mm to (126.8, 128.0), turned to 90 degrees
- moved C49 90.8 mm to (120.9, 136.4), turned to 90 degrees
- moved C52 90.1 mm to (126.3, 124.3), turned to 90 degrees
- moved C54 90.0 mm to (122.7, 132.2), turned to 90 degrees
- moved C48 87.3 mm to (117.9, 136.4), turned to 90 degrees
- moved C51 86.9 mm to (120.2, 132.2), turned to 90 degrees
- moved C50 83.8 mm to (117.7, 132.2), turned to 90 degrees
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
Commit message: testing2
Parts:
- moved C38 69.9 mm to (154.2, 100.2), turned to 0 degrees
- moved C47 66.8 mm to (154.2, 102.7), turned to 0 degrees
- moved C39 63.8 mm to (154.2, 105.2), turned to 0 degrees
- moved C36 61.4 mm to (134.3, 100.4), turned to 0 degrees
- moved R17 60.8 mm to (154.2, 107.7), turned to 0 degrees
- moved R18 57.8 mm to (154.2, 110.2), turned to 0 degrees
- moved C43 57.1 mm to (134.3, 103.4), turned to 0 degrees
- moved L2 56.4 mm to (144.4, 106.2), turned to 0 degrees
- moved C40 54.8 mm to (153.6, 112.5), turned to 0 degrees
- moved C44 52.9 mm to (134.3, 106.5), turned to 0 degrees
- moved C41 52.6 mm to (153.6, 114.4), turned to 0 degrees
- moved C37 48.6 mm to (134.3, 109.5), turned to 0 degrees
- moved C45 44.4 mm to (134.3, 112.5), turned to 0 degrees
- moved C42 44.2 mm to (141.7, 114.4), turned to 0 degrees
- moved U3 42.3 mm to (138.8, 114.9), turned to 0 degrees
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Routing:
- net /12V to 5V(3A)/Vout+: track 0.00 -> 16.2 mm

Commit message: Edited PCB layout
Parts:
- moved C38 69.9 mm to (87.2, 120.1), turned to 90 degrees
- moved C47 66.8 mm to (89.7, 120.1), turned to 90 degrees
- moved C39 63.8 mm to (92.2, 120.1), turned to 90 degrees
- moved C36 61.4 mm to (87.4, 139.9), turned to 90 degrees
- moved R17 60.8 mm to (94.7, 120.1), turned to 90 degrees
- moved R18 57.8 mm to (97.2, 120.1), turned to 90 degrees
- moved C43 57.1 mm to (90.4, 139.9), turned to 90 degrees
- moved L2 56.4 mm to (93.2, 129.9), turned to 90 degrees
- moved C40 54.8 mm to (99.4, 120.7), turned to 90 degrees
- moved C44 52.9 mm to (93.4, 139.9), turned to 90 degrees
- moved C41 52.6 mm to (101.4, 120.7), turned to 90 degrees
- moved C37 48.6 mm to (96.4, 139.9), turned to 90 degrees
- moved C45 44.4 mm to (99.4, 139.9), turned to 90 degrees
- moved C42 44.2 mm to (101.4, 132.6), turned to 90 degrees
- moved U3 42.3 mm to (101.9, 135.5), turned to 90 degrees
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Routing:
- net GND: track 0.00 -> 54.9 mm
- net /12V to 5V(3A)/Vout+: track 16.2 -> 0.00 mm

Commit message: Edited PCB layout
Routing:
- net GND: track 54.9 -> 67.9 mm
Changed lines of the file:
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@@
+	)
+	(segment
+		(start 189.7911 86.5186)
+		(end 185.3161 86.5186)
+		(width 0.2)
+		(layer "F.Cu")
+		(net "GND")
 	)
 	(segment
@@
 		(width 0.2)
 		(layer "F.Cu")
+		(net "GND")
+	)
+	(segment
+		(start 185.3161 86.5186)
+		(end 179.2511 80.4536)
+		(width 0.2)
+		(layer "F.Cu")
