File: src/powerDristributionBoard.kicad_pcb (KiCad board)
At the start: 2 copper layers, 150 x 100 mm, 106 parts, among them CN1 XT90_PCB_Mount_Male, CN2 XT30_PCB_Mount_Female, CN3 XT30_PCB_Mount_Female, CN4 XT30_PCB_Mount_Female, M1 CSD19534Q5A, M2 CSD19534Q5A, M3 CSD19534Q5A, M4 NTMFS4D5N08XT1G, U1 LM74910QRGERQ1, U2 LM5190RGYR_(20V-50V), U3 TPS566238RQFR, U4 TPS566238RQFR

Commit message: qrh
Parts:
- moved C36 68.8 mm to (156.2, 140.6), turned to 180 degrees
- moved C43 65.8 mm to (156.2, 137.6), turned to 180 degrees
- moved C44 63.0 mm to (156.2, 134.5), turned to 180 degrees
- moved C37 60.4 mm to (156.2, 131.5), turned to 180 degrees
- moved C45 57.9 mm to (156.2, 128.5), turned to 180 degrees
- moved C46 55.7 mm to (156.2, 125.5), turned to 180 degrees
- moved C38 53.4 mm to (136.4, 140.8), turned to 180 degrees
- moved L2 53.2 mm to (146.2, 134.8), turned to 180 degrees
- moved U3 50.8 mm to (151.8, 126.1), turned to 180 degrees
- moved C47 50.1 mm to (136.4, 138.3), turned to 180 degrees
- moved C42 47.9 mm to (148.9, 126.6), turned to 180 degrees
- moved C39 46.9 mm to (136.4, 135.8), turned to 180 degrees
- moved C58 45.9 mm to (152.7, 95.0), turned to 180 degrees
- moved C57 44.6 mm to (152.7, 98.0), turned to 180 degrees
- moved C56 43.8 mm to (152.7, 101.0), turned to 180 degrees
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Routing:
- net /12V to 3.3V(3A)/Vin+: track 0.00 -> 15.8 mm
