File: src/powerDristributionBoard.kicad_sch (KiCad schematic)
At the start: 16 parts, among them CN1 XT90_PCB_Mount_Male, CN2 XT30_PCB_Mount_Female, CN3 XT30_PCB_Mount_Female, CN4 XT30_PCB_Mount_Female

Commit message: Completed half of the PCB layout
Other:
- moved on the sheet: CN1, CN2, CN3, CN4, D2, D3, D4, D5, D6, D7, D8, F1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

Commit message: Upated parts and BOM
Parts:
- D3, D4, D5, R19, R20, R21: now left out of the parts list
Changed lines of the file:
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@@
 		(body_style 1)
 		(exclude_from_sim no)
-		(in_bom yes)
+		(in_bom no)
 		(on_board yes)
 		(in_pos_files yes)
@@
 		(body_style 1)
 		(exclude_from_sim no)
-		(in_bom yes)
+		(in_bom no)
 		(on_board yes)
 		(in_pos_files yes)
@@
 		(body_style 1)
 		(exclude_from_sim no)
-		(in_bom yes)
+		(in_bom no)
 		(on_board yes)
 		(in_pos_files yes)
@@
 		(body_style 1)
 		(exclude_from_sim no)
-		(in_bom yes)
+		(in_bom no)
 		(on_board yes)
 		(in_pos_files yes)
@@
 		(body_style 1)
 		(exclude_from_sim no)
-		(in_bom yes)
+		(in_bom no)
 		(on_board yes)
 		(in_pos_files yes)
@@
 		(body_style 1)
 		(exclude_from_sim no)
-		(in_bom yes)
-		(on_board yes)
-		(in_pos_files yes)
+		(in_bom no)
+		(on_board yes)
+		(in_pos_files yes)

Commit message: Finalized and exported BOM to project
Parts:
- D2: LCSC Part (none) -> C55382848; MPN (none) -> E7YYD; Manufacturer (none) -> Beking Optoelectronics
- R16: LCSC Part (none) -> C54921593; MPN (none) -> HRC1206J223 HNTN; Manufacturer (none) -> HWA CHN
Changed lines of the file:
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@@
+			)
+		)
+		(property "LCSC Part" "C54921593"
+			(at 69.85 91.44 0)
+			(hide yes)
+			(show_name no)
+			(do_not_autoplace no)
+			(effects
+				(font
+					(size 1.27 1.27)
+				)
+			)
+		)
+		(property "MPN" "HRC1206J223 HNTN"
+			(at 69.85 91.44 0)
+			(hide yes)
+			(show_name no)
+			(do_not_autoplace no)
+			(effects
+				(font
+					(size 1.27 1.27)
+				)
+			)
+		)
+		(property "Manufacturer" "HWA CHN"
+			(at 69.85 91.44 0)
+			(hide yes)
+			(show_name no)
+			(do_not_autoplace no)
+			(effects
+				(font
+					(size 1.27 1.27)
+				)
 			)
 		)
@@
 			(hide yes)
 			(show_name no)
+			(do_not_autoplace no)
+			(effects
+				(font
+					(size 1.27 1.27)
+				)
+			)
+		)
+		(property "LCSC Part" "C55382848"
+			(at 69.85 100.33 90)
+			(hide yes)
+			(show_name no)
+			(do_not_autoplace no)
+			(effects
+				(font
+					(size 1.27 1.27)
+				)
+			)
+		)
+		(property "MPN" "E7YYD"
+			(at 69.85 100.33 90)
+			(hide yes)
+			(show_name no)
+			(do_not_autoplace no)
+			(effects
+				(font
+					(size 1.27 1.27)
+				)
+			)
+		)
+		(property "Manufacturer" "Beking Optoelectronics"
+			(at 69.85 100.33 90)
+			(hide yes)
+			(show_name no)
